File: keyboard/matrix.kicad_sch (KiCad schematic)
At the start: 56 parts, among them SW10 SW_Push_45deg, SW11 SW_Push_45deg, SW12 SW_Push_45deg, SW13 SW_Push_45deg, SW14 SW_Push_45deg, SW15 SW_Push_45deg, SW16 SW_Push_45deg, SW17 SW_Push_45deg, SW18 SW_Push_45deg, SW19 SW_Push_45deg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

Commit message: Redo design
Parts:
- U: renamed from D27; value D_Small -> (none)
- U: renamed from SW13; value SW_Push_45deg -> (none)
- U: renamed from SW16; value SW_Push_45deg -> (none)
- U: renamed from SW6; value SW_Push_45deg -> (none)
- U: renamed from SW27; value SW_Push_45deg -> (none)
- U: renamed from D8; value D_Small -> (none)
- U: renamed from SW11; value SW_Push_45deg -> (none)
- U: renamed from SW5; value SW_Push_45deg -> (none)
- U: renamed from D21; value D_Small -> (none)
- U: renamed from D23; value D_Small -> (none)
- U: renamed from D4; value D_Small -> (none)
- U: renamed from D24; value D_Small -> (none)
- U: renamed from D19; value D_Small -> (none)
- U: renamed from D12; value D_Small -> (none)
- U: renamed from SW4; value SW_Push_45deg -> (none)
- U: renamed from SW9; value SW_Push_45deg -> (none)
- U: renamed from SW21; value SW_Push_45deg -> (none)
- U: renamed from SW22; value SW_Push_45deg -> (none)
- U: renamed from SW12; value SW_Push_45deg -> (none)
- U: renamed from SW8; value SW_Push_45deg -> (none)
- U: renamed from SW17; value SW_Push_45deg -> (none)
- U: renamed from D16; value D_Small -> (none)
- U: renamed from D3; value D_Small -> (none)
- U: renamed from D6; value D_Small -> (none)
- U: renamed from D17; value D_Small -> (none)
- U: renamed from SW15; value SW_Push_45deg -> (none)
- U: renamed from D13; value D_Small -> (none)
- U: renamed from D11; value D_Small -> (none)
- U: renamed from D7; value D_Small -> (none)
- U: renamed from D2; value D_Small -> (none)
- U: renamed from SW19; value SW_Push_45deg -> (none)
- U: renamed from SW7; value SW_Push_45deg -> (none)
- U: renamed from D18; value D_Small -> (none)
- U: renamed from D15; value D_Small -> (none)
- U: renamed from SW20; value SW_Push_45deg -> (none)
- U: renamed from SW10; value SW_Push_45deg -> (none)
- U: renamed from D25; value D_Small -> (none)
- U: renamed from D5; value D_Small -> (none)
- U: renamed from SW18; value SW_Push_45deg -> (none)
- U: renamed from D22; value D_Small -> (none)
- U: renamed from D28; value D_Small -> (none)
- U: renamed from SW28; value SW_Push_45deg -> (none)
- U: renamed from D20; value D_Small -> (none)
- U: renamed from D26; value D_Small -> (none)
- U: renamed from SW24; value SW_Push_45deg -> (none)
- U: renamed from SW26; value SW_Push_45deg -> (none)
- U: renamed from SW3; value SW_Push_45deg -> (none)
- U: renamed from D10; value D_Small -> (none)
- U: renamed from SW23; value SW_Push_45deg -> (none)
- U: renamed from SW2; value SW_Push_45deg -> (none)
- U: renamed from SW14; value SW_Push_45deg -> (none)
- U: renamed from SW25; value SW_Push_45deg -> (none)
- U: renamed from D9; value D_Small -> (none)
- U: renamed from D14; value D_Small -> (none)
- renumbered SW1 to U, D1 to U
Other:
- title: (none) -> rkb1
